File: board/leds.kicad_sch (KiCad schematic)
At the start: 123 parts

Commit message: v2 concept: add an rp2040, microphone, usb port; rotate entire design 1/12 turn to help align usb port and led data in; rough layout
Parts:
- renumbered D1 to D124, D2 to D125, D3 to D126, D4 to D127, D5 to D128, D6 to D129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
